File: GrandPapa_Board/grandpapa_Charge.kicad_sch (KiCad schematic)
At the start: 23 parts, among them J1 3.7V LiPo Single Cell, U3 MCP73871T-1CCI/ML, U4 INA180

Commit message: Add footprints, inductors TBD
Parts:
- C10, C11, C9: footprint (none) -> Capacitor_SMD:C_0805_2012Metric_Pad1.18x1.45mm_HandSolder
- D6, D7, D8: footprint (none) -> LED_SMD:LED_1206_3216Metric_Pad1.42x1.75mm_HandSolder
- F3: footprint (none) -> Fuse:Fuse_0805_2012Metric_Pad1.15x1.40mm_HandSolder
- R20, R21, R22, R24, R4, R5, R6, TH1: footprint (none) -> Resistor_SMD:R_0805_2012Metric_Pad1.20x1.40mm_HandSolder
- TP1, TP2: footprint (none) -> Connector_PinHeader_2.54mm:PinHeader_1x01_P2.54mm_Vertical
- U4: footprint (none) -> Package_TO_SOT_SMD:SOT-23-5_HandSoldering
Changed lines of the file:
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@@
     (property "Reference" "R22" (id 0) (at 158.75 66.294 90))
     (property "Value" "0" (id 1) (at 158.75 67.818 90))
-    (property "Footprint" "" (id 2) (at 158.75 69.85 0)
+    (property "Footprint" "Resistor_SMD:R_0805_2012Metric_Pad1.20x1.40mm_HandSolder" (id 2) (at 158.75 69.85 0)
       (effects (font (size 1.27 1.27)) hide)
     )
@@
       (effects (font (size 1.27 1.27)) (justify left))
     )
-    (property "Footprint" "" (id 2) (at 134.9248 78.74 0)
+    (property "Footprint" "Capacitor_SMD:C_0805_2012Metric_Pad1.18x1.45mm_HandSolder" (id 2) (at 134.9248 78.74 0)
       (effects (font (size 1.27 1.27)) hide)
     )
@@
       (effects (font (size 1.27 1.27)) (justify left))
     )
-    (property "Footprint" "" (id 2) (at 48.895 100.965 0)
+    (property "Footprint" "Resistor_SMD:R_0805_2012Metric_Pad1.20x1.40mm_HandSolder" (id 2) (at 48.895 100.965 0)
       (effects (font (size 1.27 1.27)) hide)
     )
@@
       (effects (font (size 1.27 1.27)) (justify left))
     )
-    (property "Footprint" "" (id 2) (at 162.56 113.03 0)
+    (property "Footprint" "Resistor_SMD:R_0805_2012Metric_Pad1.20x1.40mm_HandSolder" (id 2) (at 162.56 113.03 0)
       (effects (font (size 1.27 1.27)) hide)
     )
@@
     (property "Reference" "U4" (id 0) (at 226.695 102.235 0))
     (property "Value" "INA180" (id 1) (at 226.695 104.775 0))
-    (property "Footprint" "" (id 2) (at 228.6 92.71 0)
+    (property "Footprint" "Package_TO_SOT_SMD:SOT-23-5_HandSoldering" (id 2) (at 228.6 92.71 0)
       (effects (font (size 1.27 1.27)) hide)
     )
@@
     (property "Reference" "F3" (id 0) (at 191.77 104.14 0))
     (property "Value" "1.2A" (id 1) (at 192.405 106.045 0))
-    (property "Footprint" "" (id 2) (at 186.69 99.695 0)
+    (property "Footprint" "Fuse:Fuse_0805_2012Metric_Pad1.15x1.40mm_HandSolder" (id 2) (at 186.69 99.695 0)
       (effects (font (size 1.27 1.27)) (justify left) hide)
     )
@@
     (property "Reference" "D6" (id 0) (at 121.285 122.555 90))
     (property "Value" "QBLP650-IW" (id 1) (at 126.365 124.46 90))
-    (property "Footprint" "" (id 2) (at 118.11 123.19 0)
+    (property "Footprint" "LED_SMD:LED_1206_3216Metric_Pad1.42x1.75mm_HandSolder" (id 2) (at 118.11 123.19 0)
       (effects (font (size 1.27 1.27)) hide)
     )
@@
       (effects (font (size 1.27 1.27)) (justify left))
     )
-    (property "Footprint" "" (id 2) (at 177.8 68.58 0)
+    (property "Footprint" "Connector_PinHeader_2.54mm:PinHeader_1x01_P2.54mm_Vertical" (id 2) (at 177.8 68.58 0)
       (effects (font (size 1.27 1.27)) hide)
     )
@@
       (effects (font (size 1.27 1.27)) (justify left))
     )
-    (property "Footprint" "" (id 2) (at 118.11 113.03 0)
+    (property "Footprint" "Resistor_SMD:R_0805_2012Metric_Pad1.20x1.40mm_HandSolder" (id 2) (at 118.11 113.03 0)
       (effects (font (size 1.27 1.27)) hide)
     )
@@
     (property "Reference" "D8" (id 0) (at 165.735 121.285 90))
     (property "Value" "150120BS75000" (id 1) (at 171.45 123.19 90))
-    (property "Footprint" "" (id 2) (at 162.56 123.19 0)
+    (property "Footprint" "LED_SMD:LED_1206_3216Metric_Pad1.42x1.75mm_HandSolder" (id 2) (at 162.56 123.19 0)
       (effects (font (size 1.27 1.27)) hide)
     )
@@
     (property "Reference" "D7" (id 0) (at 148.209 122.047 90))
     (property "Value" "156120RS75000" (id 1) (at 141.605 123.825 90))
-    (property "Footprint" "" (id 2) (at 151.13 123.19 0)
+    (property "Footprint" "LED_SMD:LED_1206_3216Metric_Pad1.42x1.75mm_HandSolder" (id 2) (at 151.13 123.19 0)
       (effects (font (size 1.27 1.27)) hide)
     )
@@
       (effects (font (size 1.27 1.27)) (justify left))
     )
-    (property "Footprint" "" (id 2) (at 151.13 113.03 0)
+    (property "Footprint" "Resistor_SMD:R_0805_2012Metric_Pad1.20x1.40mm_HandSolder" (id 2) (at 151.13 113.03 0)
       (effects (font (size 1.27 1.27)) hide)
     )
@@
       (effects (font (size 1.27 1.27)) (justify left))
     )
-    (property "Footprint" "" (id 2) (at 39.37 98.425 0)
+    (property "Footprint" "Resistor_SMD:R_0805_2012Metric_Pad1.20x1.40mm_HandSolder" (id 2) (at 39.37 98.425 0)
       (effects (font (size 1.27 1.27)) hide)
     )
@@
     (property "Reference" "R24" (id 0) (at 231.14 66.294 90))
     (property "Value" "0" (id 1) (at 231.14 67.818 90))
-    (property "Footprint" "" (id 2) (at 231.14 69.85 0)
+    (property "Footprint" "Resistor_SMD:R_0805_2012Metric_Pad1.20x1.40mm_HandSolder" (id 2) (at 231.14 69.85 0)
       (effects (font (size 1.27 1.27)) hide)
     )
@@
       (effects (font (size 1.27 1.27)) (justify left))
     )
-    (property "Footprint" "" (id 2) (at 62.865 64.77 0)
+    (property "Footprint" "Connector_PinHeader_2.54mm:PinHeader_1x01_P2.54mm_Vertical" (id 2) (at 62.865 64.77 0)
       (effects (font (size 1.27 1.27)) hide)
     )
@@
       (effects (font (size 1.27 1.27)) (justify left))
     )
-    (property "Footprint" "" (id 2) (at 170.4848 97.79 0)
+    (property "Footprint" "Capacitor_SMD:C_0805_2012Metric_Pad1.18x1.45mm_HandSolder" (id 2) (at 170.4848 97.79 0)
       (effects (font (size 1.27 1.27)) hide)
     )
@@
     (property "Reference" "TH1" (id 0) (at 62.23 104.14 90))
     (property "Value" "10k" (id 1) (at 62.23 106.68 90))
-    (property "Footprint" "" (id 2) (at 64.77 100.33 0)
+    (property "Footprint" "Resistor_SMD:R_0805_2012Metric_Pad1.20x1.40mm_HandSolder" (id 2) (at 64.77 100.33 0)
       (effects (font (size 1.27 1.27)) hide)
     )
@@
       (effects (font (size 1.27 1.27)) (justify left))
     )
-    (property "Footprint" "" (id 2) (at 65.0748 74.93 0)
-      (effects (font (size 1.27 1.27)) hide)
-    )
+    (property "Footprint" "Capacitor_SMD:C_0805_2012Metric_Pad1.18x1.45mm_HandSolder" (id 2) (at 65.0748 74.93 0)
+      (effects (font (size 1.27 1.27)) hide)
+    )

Commit message: change stackup, mounting holes, connector footprints, power reg layout, fuse values
Parts:
- F3: value 1.2A -> 1.5A
Changed lines of the file:
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@@
     (in_bom yes) (on_board yes)
     (property "Reference" "F3" (id 0) (at 191.77 104.14 0))
-    (property "Value" "1.2A" (id 1) (at 192.405 106.045 0))
+    (property "Value" "1.5A" (id 1) (at 192.405 106.045 0))
     (property "Footprint" "Fuse:Fuse_0805_2012Metric_Pad1.15x1.40mm_HandSolder" (id 2) (at 186.69 99.695 0)
       (effects (font (size 1.27 1.27)) (justify left) hide)

Commit message: Fix silkscreen; add logo
Parts:
- removed TP5: TestPoint, Connector_PinHeader_2.54mm:PinHeader_1x01_P2.54mm_Vertical, symbol Connector:TestPoint
Changed lines of the file:
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@@
 (kicad_sch (version 20211123) (generator eeschema)
   (paper "A4")
-  (junction (at 240.03 69.85) (diameter 0) (color 0 0 0 0)
-  )
   (junction (at 215.9 69.85) (diameter 0) (color 0 0 0 0)
   )
@@
     (stroke (width 0) (type default) (color 0 0 0 0))
   )
-  (wire (pts (xy 240.03 68.58) (xy 240.03 69.85))
-    (stroke (width 0) (type default) (color 0 0 0 0))
-  )
   (wire (pts (xy 187.96 87.63) (xy 187.96 100.965))
     (stroke (width 0) (type default) (color 0 0 0 0))
@@
     (stroke (width 0) (type default) (color 0 0 0 0))
   )
-  (wire (pts (xy 240.03 69.85) (xy 264.16 69.85))
-    (stroke (width 0) (type default) (color 0 0 0 0))
-  )
   (wire (pts (xy 56.515 100.33) (xy 56.515 119.38))
     (stroke (width 0) (type default) (color 0 0 0 0))
@@
     (stroke (width 0) (type default) (color 0 0 0 0))
   )
-  (wire (pts (xy 233.68 69.85) (xy 240.03 69.85))
+  (wire (pts (xy 233.68 69.85) (xy 264.16 69.85))
     (stroke (width 0) (type default) (color 0 0 0 0))
   )
@@
     (pin "2")
   )
-  (symbol (lib_id "Connector:TestPoint") (at 240.03 68.58 0) (unit 1)
-    (in_bom yes) (on_board yes)
-    (property "Reference" "TP5" (id 0) (at 238.252 61.722 0)
-      (effects (font (size 1.27 1.27)) (justify left))
-    )
-    (property "Value" "TestPoint" (id 1) (at 235.458 63.5 0)
-      (effects (font (size 1.27 1.27)) (justify left))
-    )
-    (property "Footprint" "Connector_PinHeader_2.54mm:PinHeader_1x01_P2.54mm_Vertical" (id 2) (at 245.11 68.58 0)
-      (effects (font (size 1.27 1.27)) hide)
-    )
-    (property "Datasheet" "~" (id 3) (at 245.11 68.58 0)
-      (effects (font (size 1.27 1.27)) hide)
-    )
-    (pin "1")
-  )
   (symbol (lib_id "Device:C") (at 66.04 71.12 0) (mirror y) (unit 1)
