File: Dev_Board_Adapter/Dev_Board_Adapter.kicad_pcb (KiCad board)
At the start: 2 copper layers, 24.7 x 28.1 mm, 4 parts, among them J1 HARWIN_KALMAN, J2 Conn_02x10_Odd_Even, J3 Conn_01x03_Male, J4 Conn_01x08_Male

Commit message: Add logo n stuff; front pour
Parts:
- added G***: LOGO, Dev_Board_Adpater:Logo_SilkScreen_5mm, F.Cu at (116.8, 72.9)
- J4: moved to B.Cu
- turned J4 to 0 degrees
Routing:
- added copper zone on F.Cu, net GND
Other:
- board text added: "2022-12-09"
- board text added: "J. Dolina"
- board text added: "Paid Sick Day"
- board text added: "v1.0"

Commit message: gerbers, take 2
Parts:
- turned J1 to 90 degrees
Routing:
- net +5V: track 26.9 -> 33.3 mm
- net /CAN_PAYLOAD+: track 15.9 -> 20.2 mm
- net /CAN_PAYLOAD-: track 15.9 -> 15.2 mm
Changed lines of the file:
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@@
   (setup
     (pad_to_mask_clearance 0)
-    (grid_origin 129.54 73.406)
+    (grid_origin 129.794 75.184)
     (pcbplotparams
-      (layerselection 0x00010fc_ffffffff)
+      (layerselection 0x00010f0_ffffffff)
       (disableapertmacros false)
       (usegerberextensions false)
@@
       (usegerberadvancedattributes true)
       (creategerberjobfile true)
+      (gerberprecision 5)
       (svguseinch false)
       (svgprecision 6)
@@
       (outputformat 1)
       (mirror false)
-      (drillshape 1)
+      (drillshape 0)
       (scaleselection 1)
-      (outputdirectory "")
+      (outputdirectory "gerbers/")
     )
   )
@@
     (property "Sheetname" "")
     (attr through_hole)
-    (fp_text reference "J3" (at -2.54 -0.762 180) (layer "F.SilkS")
+    (fp_text reference "J3" (at -2.54 -1.016 180) (layer "F.SilkS")
       (effects (font (size 1 1) (thickness 0.15)))
     )
@@
   )
   (footprint "Dev_Board_Adpater:connector_Harwin_M80-5000642" (layer "F.Cu")
-    (at 132.35 86.328 -90)
+    (at 132.35 86.328 90)
     (property "Sheetfile" "Dev_Board_Adapter.kicad_sch")
     (property "Sheetname" "")
     (attr through_hole)
-    (fp_text reference "J1" (at -0.222 -3.032 180) (layer "F.SilkS")
+    (fp_text reference "J1" (at -0.222 -3.032) (layer "F.SilkS")
       (effects (font (size 1 1) (thickness 0.15)))
     )
@@
     (fp_line (start 8 -2) (end -8 -2) (layer "F.SilkS") (width 0.15))
     (fp_line (start 8 2) (end 8 -2) (layer "F.SilkS") (width 0.15))
-    (pad "" np_thru_hole circle locked (at 5.5 0 270) (size 2.2 2.2) (drill 2.2) (layers *.Cu *.Mask))
-    (pad "" np_thru_hole circle locked (at -5.5 0 270) (size 2.2 2.2) (drill 2.2) (layers *.Cu *.Mask))
-    (pad "1" thru_hole rect locked (at -2 1 270) (size 1.2 1.2) (drill 0.68) (layers *.Cu *.Mask)
+    (pad "" np_thru_hole circle locked (at 5.5 0 90) (size 2.2 2.2) (drill 2.2) (layers *.Cu *.Mask))
+    (pad "" np_thru_hole circle locked (at -5.5 0 90) (size 2.2 2.2) (drill 2.2) (layers *.Cu *.Mask))
+    (pad "1" thru_hole rect locked (at -2 1 90) (size 1.2 1.2) (drill 0.68) (layers *.Cu *.Mask)
       (net 29 "unconnected-(J1-Pad1)") (pinfunction "Pin_1") (pintype "passive+no_connect"))
-    (pad "2" thru_hole circle locked (at 0 1 270) (size 1.2 1.2) (drill 0.68) (layers *.Cu *.Mask)
+    (pad "2" thru_hole circle locked (at 0 1 90) (size 1.2 1.2) (drill 0.68) (layers *.Cu *.Mask)
       (net 22 "+5V") (pinfunction "Pin_2") (pintype "passive"))
-    (pad "3" thru_hole circle locked (at 2 1 270) (size 1.2 1.2) (drill 0.68) (layers *.Cu *.Mask)
+    (pad "3" thru_hole circle locked (at 2 1 90) (size 1.2 1.2) (drill 0.68) (layers *.Cu *.Mask)
       (net 21 "GND") (pinfunction "Pin_3") (pintype "passive"))
-    (pad "4" thru_hole circle locked (at -2 -1 270) (size 1.2 1.2) (drill 0.68) (layers *.Cu *.Mask)
+    (pad "4" thru_hole circle locked (at -2 -1 90) (size 1.2 1.2) (drill 0.68) (layers *.Cu *.Mask)
       (net 31 "/CAN_PAYLOAD+") (pinfunction "Pin_4") (pintype "passive"))
-    (pad "5" thru_hole circle locked (at 0 -1 270) (size 1.2 1.2) (drill 0.68) (layers *.Cu *.Mask)
+    (pad "5" thru_hole circle locked (at 0 -1 90) (size 1.2 1.2) (drill 0.68) (layers *.Cu *.Mask)
       (net 30 "/CAN_PAYLOAD-") (pinfunction "Pin_5") (pintype "passive"))
-    (pad "6" thru_hole circle locked (at 2 -1 270) (size 1.2 1.2) (drill 0.68) (layers *.Cu *.Mask))
+    (pad "6" thru_hole circle locked (at 2 -1 90) (size 1.2 1.2) (drill 0.68) (layers *.Cu *.Mask))
   )
   (footprint "Dev_Board_Adpater:Logo_SilkScreen_5mm" (layer "F.Cu")
@@
     (style (thickness 0.15) (arrow_length 1.27) (text_position_mode 2) (extension_height 0.58642) (extension_offset 0.5) keep_text_aligned)
   )
-  (segment (start 128.778 86.868) (end 129.318 86.328) (width 1) (layer "F.Cu") (net 22))
+  (segment (start 120.396 92.964) (end 120.396 95.504) (width 1) (layer "F.Cu") (net 22))
+  (segment (start 135.382 96.266) (end 135.382 87.122) (width 1) (layer "F.Cu") (net 22))
+  (segment (start 135.382 87.122) (end 134.588 86.328) (width 1) (layer "F.Cu") (net 22))
+  (segment (start 121.412 96.52) (end 135.128 96.52) (width 1) (layer "F.Cu") (net 22))
+  (segment (start 119.4308 91.9988) (end 120.396 92.964) (width 1) (layer "F.Cu") (net 22))
   (segment (start 120.396 95.504) (end 121.412 96.52) (width 1) (layer "F.Cu") (net 22))
-  (segment (start 128.778 95.504) (end 128.778 86.868) (width 1) (layer "F.Cu") (net 22))
+  (segment (start 134.588 86.328) (end 133.35 86.328) (width 1) (layer "F.Cu") (net 22))
   (segment (start 117.0686 91.9988) (end 119.4308 91.9988) (width 1) (layer "F.Cu") (net 22))
-  (segment (start 120.396 92.964) (end 120.396 95.504) (width 1) (layer "F.Cu") (net 22))
-  (segment (start 119.4308 91.9988) (end 120.396 92.964) (width 1) (layer "F.Cu") (net 22))
-  (segment (start 121.412 96.52) (end 127.762 96.52) (width 1) (layer "F.Cu") (net 22))
-  (segment (start 127.762 96.52) (end 128.778 95.504) (width 1) (layer "F.Cu") (net 22))
-  (segment (start 129.318 86.328) (end 131.35 86.328) (width 1) (layer "F.Cu") (net 22))
-  (segment (start 131.191 75.438) (end 130.302 75.438) (width 0.2) (layer "F.Cu") (net 30))
-  (segment (start 130.302 75.438) (end 129.54 74.676) (width 0.2) (layer "F.Cu") (net 30))
-  (segment (start 134.366 78.613) (end 131.191 75.438) (width 0.2) (layer "F.Cu") (net 30))
-  (segment (start 134.366 85.312) (end 134.366 78.613) (width 0.2) (layer "F.Cu") (net 30))
-  (segment (start 129.54 74.676) (end 129.54 73.406) (width 0.2) (layer "F.Cu") (net 30))
-  (segment (start 133.35 86.328) (end 134.366 85.312) (width 0.2) (layer "F.Cu") (net 30))
-  (segment (start 133.95 78.762006) (end 133.95 83.728) (width 0.2) (layer "F.Cu") (net 31))
-  (segment (start 130.81 76.2) (end 131.387994 76.2) (width 0.2) (layer "F.Cu") (net 31))
-  (segment (start 131.387994 76.2) (end 133.95 78.762006) (width 0.2) (layer "F.Cu") (net 31))
-  (segment (start 133.95 83.728) (end 133.35 84.328) (width 0.2) (layer "F.Cu") (net 31))
-  (via (at 130.81 76.2) (size 0.8) (drill 0.4) (layers "F.Cu" "B.Cu") (free) (net 31))
-  (segment (start 130.81 76.2) (end 130.81 75.692) (width 0.2) (layer "B.Cu") (net 31))
-  (segment (start 131.318 75.184) (end 133.858 75.184) (width 0.2) (layer "B.Cu") (net 31))
-  (segment (start 130.81 75.692) (end 131.318 75.184) (width 0.2) (layer "B.Cu") (net 31))
-  (segment (start 133.858 75.184) (end 134.62 74.422) (width 0.2) (layer "B.Cu") (net 31))
-  (segment (start 134.62 74.422) (end 134.62 73.406) (width 0.2) (layer "B.Cu") (net 31))
+  (segment (start 135.128 96.52) (end 135.382 96.266) (width 1) (layer "F.Cu") (net 22))
+  (segment (start 129.54 77.724) (end 129.54 83.790102) (width 0.2) (layer "F.Cu") (net 30))
+  (segment (start 129.54 73.406) (end 129.54 75.184) (width 0.2) (layer "F.Cu") (net 30))
+  (segment (start 129.54 75.184) (end 129.794 75.438) (width 0.2) (layer "F.Cu") (net 30))
+  (segment (start 131.35 85.600102) (end 131.35 86.328) (width 0.2) (layer "F.Cu") (net 30))
+  (segment (start 130.556 75.438) (end 130.81 75.692) (width 0.2) (layer "F.Cu") (net 30))
+  (segment (start 129.794 75.438) (end 130.556 75.438) (width 0.2) (layer "F.Cu") (net 30))
+  (segment (start 129.54 83.790102) (end 131.35 85.600102) (width 0.2) (layer "F.Cu") (net 30))
+  (segment (start 130.81 76.454) (end 129.54 77.724) (width 0.2) (layer "F.Cu") (net 30))
+  (segment (start 130.81 75.692) (end 130.81 76.454) (width 0.2) (layer "F.Cu") (net 30))
+  (segment (start 130.9 87.435051) (end 130.9 87.878) (width 0.2) (layer "F.Cu") (net 31))
+  (segment (start 129.14048 85.675531) (end 130.9 87.435051) (width 0.2) (layer "F.Cu") (net 31))
+  (segment (start 129.794 76.2) (end 129.14048 76.85352) (width 0.2) (layer "F.Cu") (net 31))
+  (segment (start 131.35 88.328) (end 130.9 87.878) (width 0.2) (layer "F.Cu") (net 31))
+  (segment (start 129.14048 76.85352) (end 129.14048 85.675531) (width 0.2) (layer "F.Cu") (net 31))
+  (via (at 129.794 76.2) (size 0.8) (drill 0.4) (layers "F.Cu" "B.Cu") (free) (net 31))
+  (segment (start 134.62 74.93) (end 134.62 73.406) (width 0.2) (layer "B.Cu") (net 31))
+  (segment (start 130.556 75.438) (end 134.112 75.438) (width 0.2) (layer "B.Cu") (net 31))
+  (segment (start 134.112 75.438) (end 134.62 74.93) (width 0.2) (layer "B.Cu") (net 31))
+  (segment (start 129.794 76.2) (end 130.556 75.438) (width 0.2) (layer "B.Cu") (net 31))
   (zone (net 21) (net_name "GND") (layer "F.Cu") (hatch edge 0.508)
     (connect_pads (clearance 0.508))
